File: firmware/hardware/aquasentinel-hardware.kicad_pcb (KiCad board)
At the start: 2 copper layers, 13 parts, among them J1 5V_BOOST_OUT, J2 1S_LIION_BAT, J3 BAT_LEVEL_LED, J4 ESP32_CAM_USED_PINS, J5 STM32F103C8T6_BLUEPILL_USED_P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, J6 SERVO_PAN_SG90, J7 SERVO_TILT_SG90, J8 SSD1306_OLED_I2C, SW1 USER_HOME_CALIB

Commit message: chore(hardware): 更新原理图封装与ERC报告
Parts:
- J4: value ESP32_CAM_USED_PINS -> ESP32-CAM; footprint Connector_PinHeader_2.54mm:PinHeader_1x04_P2.54mm_Vertical -> AquaSentinelFootprints:ESP32_CAM_AI_Thinker_2x08_P22.86mm_Vertical_Labeled
- J5: value STM32F103C8T6_BLUEPILL_USED_PINS -> STM32F103C8T6_BLUEPILL; footprint Connector_PinSocket_2.54mm:PinSocket_2x20_P2.54mm_Vertical -> AquaSentinelFootprints:STM32_BluePill_2x20_P17.78mm_Vertical_Labeled
- J8: footprint Connector_PinSocket_2.54mm:PinSocket_2x08_P2.54mm_Vertical -> Connector_PinHeader_2.54mm:PinHeader_1x04_P2.54mm_Vertical
- SW1: footprint Button_Switch_THT:SW_PUSH_6mm -> AquaSentinelFootprints:SW_PUSH_6mm_2Pin_LR
- moved J7 72.7 mm to (89.0, 88.5)
- moved J2 69.0 mm to (90.0, 125.0)
- moved J6 64.7 mm to (89.0, 76.0)
- moved SW1 63.6 mm to (85.7, 109.5)
- moved J3 62.2 mm to (102.0, 125.2)
- moved R1 56.8 mm to (113.7, 131.0)
- moved J1 41.5 mm to (132.1, 63.5)
- moved R2 39.4 mm to (139.8, 130.5), turned to 180 degrees
- moved J8 36.8 mm to (114.3, 55.9), turned to -90 degrees
- moved C2 33.9 mm to (135.8, 103.5)
- moved J5 27.6 mm to (111.4, 67.3)
- moved C1 25.2 mm to (135.5, 116.0)
- moved J4 19.0 mm to (156.8, 107.2), turned to 180 degrees
Connections:
- J4 pad 2: /GND -> unconnected-(J4-3V3-Pad2)
- J4 pad 3: /UART_ESP_TX -> /GND
- J4 pad 4: /UART_ESP_RX -> unconnected-(J4-IO16-Pad4)
- J5 pad 1: /VCC_5V -> unconnected-(J5-VBAT-Pad1)
- J5 pad 10: /BTN_USER -> unconnected-(J5-PB8-Pad10)
- J5 pad 11: /BAT_SENSE -> unconnected-(J5-PA1-Pad11)
- J5 pad 12: (no net) -> /I2C_SDA
- J5 pad 13: (no net) -> unconnected-(J5-PA2-Pad13)
- J5 pad 14: (no net) -> /I2C_SCL
- J5 pad 15: (no net) -> unconnected-(J5-PA3-Pad15)
- J5 pad 16: (no net) -> unconnected-(J5-PB5-Pad16)
- J5 pad 17: (no net) -> unconnected-(J5-PA4-Pad17)
- J5 pad 18: (no net) -> unconnected-(J5-PB4-Pad18)
- J5 pad 19: (no net) -> unconnected-(J5-PA5-Pad19)
- J5 pad 2: /GND -> /VCC_3V3
- J5 pad 20: (no net) -> unconnected-(J5-PB3-Pad20)
- J5 pad 21: (no net) -> /SERVO_PAN
- J5 pad 22: (no net) -> unconnected-(J5-PA15-Pad22)
- J5 pad 23: (no net) -> /SERVO_TILT
- J5 pad 24: (no net) -> unconnected-(J5-PA12-Pad24)
- J5 pad 25: (no net) -> unconnected-(J5-PB0-Pad25)
- J5 pad 26: (no net) -> unconnected-(J5-PA11-Pad26)
- J5 pad 27: (no net) -> unconnected-(J5-PB1-Pad27)
- J5 pad 28: (no net) -> /UART_ESP_TX
- J5 pad 29: (no net) -> unconnected-(J5-PB10-Pad29)
- J5 pad 3: /VCC_3V3 -> unconnected-(J5-PC13-Pad3)
- J5 pad 30: (no net) -> /UART_ESP_RX
- J5 pad 31: (no net) -> unconnected-(J5-PB11-Pad31)
- J5 pad 32: (no net) -> unconnected-(J5-PA8-Pad32)
- J5 pad 33: (no net) -> unconnected-(J5-NRST-Pad33)
- J5 pad 34: (no net) -> unconnected-(J5-PB15-Pad34)
- J5 pad 35: (no net) -> unconnected-(J5-3V3-Pad35)
- J5 pad 36: (no net) -> unconnected-(J5-PB14-Pad36)
- J5 pad 37: (no net) -> /GND
- J5 pad 38: (no net) -> unconnected-(J5-PB13-Pad38)
- J5 pad 39: (no net) -> unconnected-(J5-GND-Pad39)
- J5 pad 4: /UART_ESP_TX -> /GND
- J5 pad 40: (no net) -> /BTN_USER
- J5 pad 5: /UART_ESP_RX -> unconnected-(J5-PC14-Pad5)
- J5 pad 6: /SERVO_PAN -> /VCC_5V
- J5 pad 7: /SERVO_TILT -> unconnected-(J5-PC15-Pad7)
- J5 pad 8: /I2C_SCL -> unconnected-(J5-PB9-Pad8)
- J5 pad 9: /I2C_SDA -> /BAT_SENSE
Routing:
- net /VCC_5V: track 20.1 -> 0.18 mm
- net /GND: track 9.33 -> 0.00 mm
- net /BAT_SENSE: track 9.30 -> 0.00 mm
