File: firmware/hardware/aquasentinel-hardware.kicad_sch (KiCad schematic)
At the start: 13 parts, among them J1 5V_BOOST_OUT, J2 1S_LIION_BAT, J3 BAT_LEVEL_LED, J4 ESP32_CAM_AI_THINKER, J5 STM32F103C8T6_BLUEPILL, J6 SERVO_PAN_SG90, J7 SERVO_TILT_SG90, J8 SSD1306_OLED_I2C, SW1 USER_HOME_CALIB

Commit message: chore(hardware): 更新原理图封装与ERC报告
Parts:
- J4: value ESP32_CAM_AI_THINKER -> ESP32-CAM; footprint AquaSentinelFootprints:ESP32_CAM_AI_Thinker_2x08_P22.86mm_Vertical -> AquaSentinelFootprints:ESP32_CAM_AI_Thinker_2x08_P22.86mm_Vertical_Labeled
- J5: footprint AquaSentinelFootprints:STM32_BluePill_2x20_P17.78mm_Vertical -> AquaSentinelFootprints:STM32_BluePill_2x20_P17.78mm_Vertical_Labeled
- J8: footprint Connector_PinSocket_2.54mm:PinSocket_2x08_P2.54mm_Vertical -> Connector_PinHeader_2.54mm:PinHeader_1x04_P2.54mm_Vertical
- SW1: footprint Button_Switch_THT:SW_PUSH_6mm -> AquaSentinelFootprints:SW_PUSH_6mm_2Pin_LR
Connections:
- net BAT_SENSE: now also J5.9 (PA0_/_ADC_IN0)
- net BTN_USER: now also J5.40 (PB12)
- net GND: now also J4.3 (GND), J5.37 (GND), J5.4 (GND)
- net I2C_SCL: now also J5.14 (PB6_/_I2C1_SCL)
- net I2C_SDA: now also J5.12 (PB7_/_I2C1_SDA)
- net SERVO_PAN: now also J5.21 (PA6_/_TIM3_CH1)
- net SERVO_TILT: now also J5.23 (PA7_/_TIM3_CH2)
- net UART_ESP_RX: now also J4.11 (IO14), J5.30 (PA9_/_USART1_TX)
- net UART_ESP_TX: now also J4.7 (IO13), J5.28 (PA10_/_USART1_RX)
- net VCC_3V3: now also J5.2 (3V3)
- net VCC_5V: now also J4.1 (5V), J5.6 (5V)
- no-connect marks 41 -> 43
